File: KiCad_Pi_Pico_Andur/Pi_Pico_Andur.kicad_sch (KiCad schematic)
At the start: 1 part

Commit message: kicad
Parts:
- added D1, D2: 1N4007, Diode_THT:D_DO-41_SOD81_P10.16mm_Horizontal, symbol Diode:1N4007
- added D3, D4: LED, symbol Device:LED
- added J1: Jack-DC, symbol Connector:Jack-DC
- added J2, J3, J4: Screw_Terminal_01x02, TerminalBlock:TerminalBlock_MaiXu_MX126-5.0-02P_1x02_P5.00mm, symbol Connector:Screw_Terminal_01x02
- added J5: Screw_Terminal_01x03, symbol Connector:Screw_Terminal_01x03
- added R1, R3, R4: 470, symbol Device:R
- added R2: 10K, symbol Device:R
- added U1: ~, symbol Tauno_Library:Tauno_OKY3504-1
- added U2: ~, symbol Tauno_Library:Tauno_Oled_096_SSD1306
- added U3, U4: ~, symbol Tauno_Library:Tauno_Rotary_Encoder
- added U5: ~, symbol Tauno_Library:Tauno_TOF_VL53LOX
- added U6: PC817, Package_DIP:DIP-4_W7.62mm, symbol Isolator:PC817
Connections:
- net GND: now reaches A1.13 (GND), A1.18 (GND), A1.23 (GND), A1.28 (GND), A1.3 (GND), A1.38 (GND), A1.8 (GND)
- net GND: now also D3.1 (K), D4.1 (K), U1.4 (OUT-), U2.1 (GND), U3.5 (GND), U4.5 (GND), U6.2
- net +3.3V: now reaches A1.36 (3V3)
- net +3.3V: now also U2.2 (VCC), U3.4 (+), U4.4 (+)
- net VSYS: now reaches A1.39 (VSYS)
- net VSYS: now also U1.3 (OUT+)
- net SDA: now reaches A1.6 (GPIO4)
- net SDA: now also U2.4 (SDA)
- net SCL: now reaches A1.7 (GPIO5)
- net SCL: now also U2.3 (SCL)
- new net: R1.2, U6.1
- new net: D4.2 (A), R4.1
- new net: D1.2 (A), D2.1 (K)
- new net: D2.2 (A), J1.1
- new net: D1.1 (K), U1.1 (IN+)
- new net: J1.2, U1.2 (IN1)
- new net: J2.1 (Pin_1), U5.1 (VIN)
- new net: J2.2 (Pin_2), U5.2 (GND)
- new net: D3.2 (A), R3.1
- new net: J4.1 (Pin_1), U5.5 (GPIO1)
- new net: J4.2 (Pin_2), U5.6 (XSHUT)
- new net: J3.1 (Pin_1), U5.3 (SCL)
- new net: J3.2 (Pin_2), U5.4 (SDA)
- new net External_GND: J5.3 (Pin_3), U6.3
- new net External_GPIO: J5.2 (Pin_2), R2.1, U6.4
- new net External_VCC: J5.1 (Pin_1), R2.2
- new net Green_LED_GPIO: R3.2
- new net Left_RE_CLK: U3.1 (CLK)
- new net Left_RE_DT: U3.2 (DT)
- new net Left_RE_SW: U3.3 (SW)
- new net Red_LED_GPIO: R4.2
- new net Right_RE_CLK: U4.1 (CLK)
- new net Right_RE_DT: U4.2 (DT)
- new net Right_RE_SW: U4.3 (SW)
- new net Signal_OUT: R1.1
Other:
- note added: "24V IN?"
- note added: "ANDUR"
- note added: "KASUTAJALIIDES"
- note added: "MAX seadistamine"
- note added: "MCU Internal PullUp?"
- note added: "MIN seadistamine"
- note added: "Pi Pico 2"
- note added: "SIGNAAL VÄLJA"
- note added: "VOOL"
- note added: "VSYS: IN 1.8V-5.5V"
- moved on the sheet: A1

Commit message: kicad update
Parts:
- U2: value ~ -> Tauno_Oled_096_SSD1306; footprint (none) -> Taunoe_footprints:Tauno_OLED_ssd1306
Connections:
- net +3.3V: now also U2.1 (VCC); no longer U2.2 (VCC)
- net GND: now also U2.2 (GND); no longer U2.1 (GND)
Changed lines of the file:
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@@
+	(wire
+		(pts
+			(xy 186.69 35.56) (xy 186.69 43.18)
+		)
+		(stroke
+			(width 0)
+			(type default)
+		)
+	)
 	(wire
 		(pts
@@
 	(wire
 		(pts
-			(xy 199.39 36.83) (xy 199.39 33.02)
-		)
-		(stroke
-			(width 0)
-			(type default)
-		)
-	)
-	(wire
-		(pts
 			(xy 246.38 78.74) (xy 246.38 81.28)
 		)
@@
 	(wire
 		(pts
-			(xy 186.69 33.02) (xy 186.69 39.37)
-		)
-		(stroke
-			(width 0)
-			(type default)
-		)
-	)
-	(wire
-		(pts
 			(xy 91.44 38.1) (xy 91.44 48.26)
 		)
@@
 	(wire
 		(pts
+			(xy 201.93 36.83) (xy 201.93 35.56)
+		)
+		(stroke
+			(width 0)
+			(type default)
+		)
+	)
+	(wire
+		(pts
 			(xy 142.24 35.56) (xy 120.65 35.56)
 		)
@@
 	(wire
 		(pts
-			(xy 201.93 31.75) (xy 201.93 36.83)
-		)
-		(stroke
-			(width 0)
-			(type default)
-		)
-	)
-	(wire
-		(pts
 			(xy 38.1 38.1) (xy 62.23 38.1)
 		)
@@
 	(wire
 		(pts
+			(xy 201.93 35.56) (xy 186.69 35.56)
+		)
+		(stroke
+			(width 0)
+			(type default)
+		)
+	)
+	(wire
+		(pts
 			(xy 271.78 38.1) (xy 271.78 40.64)
 		)
@@
 	(wire
 		(pts
-			(xy 199.39 33.02) (xy 186.69 33.02)
+			(xy 199.39 31.75) (xy 199.39 36.83)
 		)
 		(stroke
@@
 			)
 		)
-		(property "Value" "~"
+		(property "Value" "Tauno_Oled_096_SSD1306"
 			(at 214.63 50.1649 0)
 			(effects
@@
 			)
 		)
-		(property "Footprint" ""
+		(property "Footprint" "Taunoe_footprints:Tauno_OLED_ssd1306"
 			(at 201.93 48.26 0)
 			(effects
@@
 			)
 		)
-		(property "Description" ""
+		(property "Description" "Tauno_Oled_096_SSD1306"
 			(at 201.93 48.26 0)
 			(effects
@@
 	(symbol
 		(lib_id "power:GND")
-		(at 186.69 39.37 0)
+		(at 186.69 43.18 0)
 		(unit 1)
 		(exclude_from_sim no)
@@
 		(fields_autoplaced yes)
 		(property "Reference" "#PWR04"
-			(at 186.69 45.72 0)
+			(at 186.69 49.53 0)
 			(effects
 				(font
@@
 		)
 		(property "Value" "GND"
-			(at 186.69 44.45 0)
+			(at 186.69 48.26 0)
 			(effects
 				(font
@@
 		)
 		(property "Footprint" ""
-			(at 186.69 39.37 0)
+			(at 186.69 43.18 0)
 			(effects
 				(font
@@
 		)
 		(property "Datasheet" ""
-			(at 186.69 39.37 0)
+			(at 186.69 43.18 0)
 			(effects
 				(font
@@
 		)
 		(property "Description" "Power symbol creates a global label with name \"GND\" , ground"
-			(at 186.69 39.37 0)
+			(at 186.69 43.18 0)
 			(effects
 				(font
@@
 	(symbol
 		(lib_id "power:+3.3V")
-		(at 201.93 31.75 0)
+		(at 199.39 31.75 0)
 		(unit 1)
 		(exclude_from_sim no)
@@
 		(fields_autoplaced yes)
 		(property "Reference" "#PWR03"
-			(at 201.93 35.56 0)
+			(at 199.39 35.56 0)
 			(effects
 				(font
@@
 		)
 		(property "Value" "+3.3V"
-			(at 201.93 26.67 0)
+			(at 199.39 26.67 0)
 			(effects
 				(font
@@
 		)
 		(property "Footprint" ""
-			(at 201.93 31.75 0)
+			(at 199.39 31.75 0)
 			(effects
 				(font
@@
 		)
 		(property "Datasheet" ""
-			(at 201.93 31.75 0)
+			(at 199.39 31.75 0)
 			(effects
 				(font
@@
 		)
 		(property "Description" "Power symbol creates a global label with name \"+3.3V\""
-			(at 201.93 31.75 0)
-			(effects
-				(font
+			(at 199.39 31.75 0)
+			(effects
+				(font
