File: KiCad/proto_layout/proto_layout.kicad_pcb (KiCad board)
At the start: 2 copper layers, 8 parts, among them J2 Screw_Terminal_01x02, J3 Screw_Terminal_01x02, J4 Screw_Terminal_01x02, U2 Tauno_Oled_096_SSD1306, U6 PC817

Commit message: kicad files
Parts:
- added U3: ~, Taunoe_footprints:Tauno_Rotary_Encoder, F.Cu at (85.4, 129.8)
- added U4: ~, Taunoe_footprints:Tauno_Rotary_Encoder, F.Cu at (110.8, 129.8)
- moved U2 21.0 mm to (112.2, 89.2)
Connections:
- A1 pad 21: unconnected-(A1-GPIO16-Pad21) -> Left_RE_CLK
- A1 pad 22: unconnected-(A1-GPIO17-Pad22) -> Left_RE_DT
- A1 pad 24: unconnected-(A1-GPIO18-Pad24) -> Left_RE_SW
- A1 pad 25: unconnected-(A1-GPIO19-Pad25) -> Right_RE_CLK
- A1 pad 26: unconnected-(A1-GPIO20-Pad26) -> Right_RE_DT
- A1 pad 27: unconnected-(A1-GPIO21-Pad27) -> Right_RE_SW
