File: KiCad/skeem/skeem.kicad_sch (KiCad schematic)
At the start: 17 parts, among them J2 Barrel_Jack_Switch, J5 Screw_Terminal_01x03, U1 OKY3504-1, U2 VL53L01-v2, U6 PC817

Commit message: skeem
Parts:
- added ADCPINS1, J1, PINS1, PINS2, PINS3, PINS4: Screw_Terminal_01x03, symbol Connector:Screw_Terminal_01x03
- added Power1, Power2, Power3: Screw_Terminal_01x02, symbol Connector:Screw_Terminal_01x02
- added R5: 470, symbol Device:R
- added R6: 10K, symbol Device:R
- added U5: PC817, Package_DIP:DIP-4_W7.62mm, symbol Isolator:PC817
Connections:
- net +3.3V: now also PINS2.1 (Pin_1), Power1.1 (Pin_1), Power2.1 (Pin_1), Power3.1 (Pin_1)
- net GND: now also A1.33 (AGND), PINS1.3 (Pin_3), PINS2.3 (Pin_3), Power1.2 (Pin_2), Power2.2 (Pin_2), Power3.2 (Pin_2), U5.2
- net Sensor_XSHUT: now reaches A1.10 (GPIO7), U2.6 (XSHUT)
- net GPIO8: now reaches A1.11 (GPIO8)
- net GPIO8: now also PINS2.2 (Pin_2)
- net GPIO9: now reaches A1.12 (GPIO9)
- net GPIO9: now also PINS4.1 (Pin_1)
- net GPIO10: now reaches A1.14 (GPIO10)
- net GPIO10: now also PINS4.2 (Pin_2)
- net GPIO11: now reaches A1.15 (GPIO11)
- net GPIO11: now also PINS4.3 (Pin_3)
- net GPIO12: now reaches A1.16 (GPIO12)
- net GPIO12: now also PINS3.3 (Pin_3)
- net GPIO13: now reaches A1.17 (GPIO13)
- net GPIO13: now also PINS3.2 (Pin_2)
- net GPIO14: now reaches A1.19 (GPIO14)
- net GPIO14: now also PINS3.1 (Pin_1)
- net Signal_OUT_1: now reaches A1.29 (GPIO22)
- net Signal_OUT_1: now also R1.1
- net GPIO0: now reaches A1.30 (RUN)
- net GPIO0: now also PINS1.1 (Pin_1)
- net GPIO26: now reaches A1.31 (GPIO26_ADC0)
- net GPIO26: now also ADCPINS1.1 (Pin_1)
- net GPIO27: now reaches A1.32 (GPIO27_ADC1)
- net GPIO27: now also ADCPINS1.2 (Pin_2)
- net GPIO28: now reaches A1.34 (GPIO28_ADC2)
- net GPIO28: now also ADCPINS1.3 (Pin_3)
- net GPIO1: now reaches A1.37 (3V3_EN)
- net GPIO1: now also PINS1.2 (Pin_2)
- net Sensor_GPIO01: now reaches A1.9 (GPIO6), U2.5 (GPIO01)
- net External_GND renamed External_GND1
- net External_GPIO renamed External_GPIO1
- net External_VCC renamed External_VCC1
- net Signal_OUT renamed Signal_OUT_2
- net Signal_OUT_2: now also R5.1; no longer R1.1
- new net: R5.2, U5.1
- new net External_GND2: J1.3 (Pin_3), U5.3
- new net External_GPIO2: J1.2 (Pin_2), R6.1, U5.4
- new net External_VCC2: J1.1 (Pin_1), R6.2
- no-connect marks 0 -> 1
Other:
- note added: "UI"
- note removed: "GUI"
- moved on the sheet: D1, D2, D3, D4, J2, J5, R1, R2, R3, R4, U1, U2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
